File: Schematics/Nigun.sch (KiCad schematic (older format))
At the start: 136 parts, among them J1 RF_INPUT, J2 SMA, J3 SMA, J4 USB-MICRO-B, P1 CONN_02X04, P2 CONN_02X03, SW1 SW_PUSH_SMALL_H, T1 TC1-1-43A+, T2 TC1-1-43A+, T3 TC4-1W+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

Commit message: Finished schematics
Parts:
- removed C85, C88: 10uF, symbol C
- removed C86: 1uF, symbol C
- removed C87, C89: 100nF, symbol C
- removed P2: CONN_02X03, symbol CONN_02X03
- removed R1: 0, symbol R
- removed R15, R16: 68, symbol R
- removed R17: 10K, symbol R
- removed U8: SAMD20E17A-A, samd20e17a:QFN50P500X500X100-33N, symbol SAMD20E17A-A
- added C85, C89: 10uF, symbol C_Small
- added C86, C88, C90: 100nF, symbol C_Small
- added C87: 1uF, symbol C_Small
- added P2: CONN_SWD, symbol CONN_SWD
- added R15: 10k, symbol R_Small
- added R16, R17, R22, R23, R24, R25, R26, R27, R29: 0, symbol R_Small
- added R28: 10k, symbol R
- added U8: STF202, hack-footprints:TSOP-6, symbol STF202
- added U9: ATSAMD21E, symbol ATSAMD21E
- D3: value blue_led -> Blue
- D4: value blue_led -> Red
- D5: value green_led -> Green
- R14: value 10k -> 0
- R20, R21: value 1k -> 330
- R8: value 2k -> 330
Connections:
- net labels added: !RESET, ADRF_MUXOUT, ADRF_VTUNE, IN_SW_VCTL1, IN_SW_VCTL2, MCU_VDDIN, OUT_SW_V1, OUT_SW_V2, SWDCLK, SWDIO, TCXO_OUT, USB_D+, USB_D-, VDDIN
- net labels removed: +5V, 6612OUT_MUXOUT, CPOUT, OUTSW_V1, OUTSW_V2, RESET, SWIN_VCTL1, SWIN_VCTL2, USB_DM, USB_DP, VTUNE
- wire segments 341 -> 224
- no-connect marks 8 -> 4
Other:
- note added: "DEBUG PINS"
- note added: "NIGUN (MELODY)"
- note added: "NIGUN (MELODY)\n1500-3000MHz RF Down-converter"
- note added: "SWD DEBUG CONNECTOR"
- note added: "TCXO"
- note removed: "CLK"
- note removed: "Debug pads"
- note removed: "MCU \nProgramming \nport"
- note removed: "NIGUN - 1500-3000MHz RF downconverter for SDR"
- moved on the sheet: C79, C80, C81, C82, D1, D2, D3, D4, D5, L3, P1, R12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

Commit message: Updated readme.md
Parts:
- U2: footprint (none) -> Housings_DFN_QFN:QFN-12-1EP_3x3mm_Pitch0.5mm
- U4: footprint (none) -> Capacitors_SMD:C_0805
- U9: footprint (none) -> QFN32:QFN32
Changed lines of the file:
@@
 F 0 "U2" H 10150 9800 60  0000 C CNN
 F 1 "SKY13373" H 10150 10000 60  0000 C CNN
-F 2 "" H 10350 10000 60  0000 C CNN
+F 2 "Housings_DFN_QFN:QFN-12-1EP_3x3mm_Pitch0.5mm" H 10350 10000 60  0000 C CNN
 F 3 "" H 10350 10000 60  0000 C CNN
 	1    10350 10000
@@
 F 0 "U4" H 4150 9950 60  0000 C CNN
 F 1 "LP0805A1119AS" H 4200 10400 60  0000 C CNN
-F 2 "" H 4200 10300 60  0000 C CNN
+F 2 "Capacitors_SMD:C_0805" H 4200 10300 60  0000 C CNN
 F 3 "" H 4200 10300 60  0000 C CNN
 	1    4200 10300
@@
 F 0 "U9" H 12950 1100 40  0000 L CNB
 F 1 "ATSAMD21E" H 13175 1100 40  0000 L CNB
-F 2 "" H 13600 900 60  0000 C CNN
+F 2 "QFN32:QFN32" H 13600 900 60  0000 C CNN
 F 3 "" H 12950 1100 60  0000 C CNN
 F 4 "ATSAMD21E18A-MU" H 13050 1200 60  0000 C CNN "manf#"
